Commit message: modified:   README.md 	modified:   config/config_file.rviz 	modified:   config/mapper_params_online_async_local.yaml 	modified:   description/lidar.xacro 	modified:   description/robot_core.xacro 	modified:   launch/launch_sim.launch.py

File: description/lidar.xacro (robot description, xacro)
@@ -19,5 +19,5 @@
         </collision>
         <xacro:inertial_cylinder mass="0.1" length="0.04" radius="0.05">
-            <origin xyz="0.1 0.0 0.175" rpy="0 0 0"/>
+            <origin xyz="0.1 0 0.175" rpy="0 0 0"/>
         </xacro:inertial_cylinder>
     </link>

File: description/robot_core.xacro (robot description, xacro)
@@ -27,4 +27,5 @@
     </joint>
     <link name="base_footprint">
+        <origin xyz="0.0 -0.175 0.0" rpy="0.0 0.0 0.0"/>
     </link>
     <!-- CHASSIS LINK -->
@@ -32,5 +33,5 @@
         <parent link="base_link"/>
         <child link="chassis"/>
-        <origin xyz="-0.1 0 0"/>
+        <origin xyz="-0.1 0 0.0"/>
     </joint>
     <link name="chassis">
