Commit message: new file:   config/config_file_drive.rviz new file:   description/gazebo_control.xacro modified:   description/robot.urdf.xacro modified:   description/robot_core.xacro new file:   launch/launch_sim.launch.py modified:   launch/rsp.launch.py new file:   launch/rspwithrviz.launch.py

File: description/robot_core.xacro (robot description, xacro)
@@ -41,4 +41,7 @@
         </xacro:inertial_box>
     </link>
+    <gazebo reference="chassis">
+        <material>Gazebo/White</material>
+    </gazebo>
     <!-- LEFT WHEEL LINK -->
     <joint name="left_wheel_joint" type="continuous">
@@ -64,4 +67,7 @@
         </xacro:inertial_cylinder>
     </link>
+    <gazebo reference="left_wheel">
+        <material>Gazebo/Blue</material>
+    </gazebo>
     <!-- RIGHT WHEEL LINK -->
     <joint name="right_wheel_joint" type="continuous">
@@ -87,4 +93,7 @@
         </xacro:inertial_cylinder>
     </link>
+    <gazebo reference="right_wheel">
+        <material>Gazebo/Blue</material>
+    </gazebo>
     <!-- CASTER WHEEL LINK -->
     <joint name="caster_wheel_joint" type="fixed">
@@ -109,3 +118,8 @@
         </xacro:inertial_sphere>
     </link>
+    <gazebo reference="caster_wheel">
+        <material>Gazebo/Black</material>
+        <mu1 value="0.01"/>
+        <mu2 value="0.01"/>
+    </gazebo>
 </robot>

Commit message: modified:   description/robot_core.xacro 	modified:   launch/launch_sim.launch.py

File: description/robot_core.xacro (robot description, xacro)
@@ -22,10 +22,10 @@
     <!-- BASE FOOTPRINT LINK -->
     <joint name="base_footprint_joint" type="fixed">
-        <origin xyz="0.0 0.0 0.0" rpy="0.0 0.0 0.0"/>
+        <origin xyz="0.0 0.0 -0.05" rpy="0.0 0.0 0.0"/>
         <parent link="base_link"/>
         <child link="base_footprint"/>
     </joint>
     <link name="base_footprint">
-        <origin xyz="0.0 -0.175 0.0" rpy="0.0 0.0 0.0"/>
+        <origin xyz="0.0 0.0 -0.1" rpy="0.0 0.0 0.0"/>
     </link>
     <!-- CHASSIS LINK -->
