Commit message: Already nav

File: install/mok_mobile_robot/share/mok_mobile_robot/description/robot.urdf.xacro (robot description, xacro)
@@ -3,5 +3,4 @@
     <xacro:include filename="robot_core.xacro" />
     <xacro:include filename="gazebo_control.xacro" />
-    <!-- <xacro:include filename="ros2_control.xacro" /> -->
     <xacro:include filename="lidar.xacro" />
     <xacro:include filename="depth_camera.xacro"/>

File: install/mok_mobile_robot/share/mok_mobile_robot/description/robot_core.xacro (robot description, xacro)
@@ -19,12 +19,4 @@
     <!-- BASE LINK -->
     <link name="base_link">
-    </link>
-    <!-- BASE FOOTPRINT LINK -->
-    <joint name="base_footprint_joint" type="fixed">
-        <origin xyz="0.0 0.0 0.0" rpy="0.0 0.0 0.0"/>
-        <parent link="base_link"/>
-        <child link="base_footprint"/>
-    </joint>
-    <link name="base_footprint">
     </link>
     <!-- CHASSIS LINK -->
